Commit message: add lidar

File: src/my_robot/models/my_robot/model.urdf (robot description, URDF)
Before this commit: robot my_robot, 5 links, 4 joints
Links:
- removed link laser_frame
Joints:
- removed joint laser_joint
- joint caster_wheel: origin (none) -> xyz=0.6 0 -0.2 rpy=0 0 0
- joint left_wheel_joint: origin (none) -> xyz=-0.5 0.6 0 rpy=0 0 0
- joint right_wheel_joint: origin (none) -> xyz=-0.5 -0.6 0 rpy=0 0 0
